Commit message: Vision and chess ai

File: catkin_ws/src/ros_chess/urdf/chess_robot.xacro (robot description, xacro)
@@ -330,3 +330,44 @@
     <material>Gazebo/Red</material>
   </gazebo>
+   <!-- Camera -->
+  <joint type="fixed" name="camera_joint">
+    <origin xyz="0 0 0" rpy="0 -1.57 0"/>
+    <child link="camera_link"/>
+    <parent link="gripper_base_link"/>
+    <axis xyz="0 1 0" />
+  </joint>
+  <link name='camera_link'>
+    <pose>0 0 0 0 0 0</pose>
+    <inertial>
+      <mass value="0.1"/>
+      <origin xyz="0 0 0" rpy="0 0 0"/>
+      <inertia
+          ixx="1e-6" ixy="0" ixz="0"
+          iyy="1e-6" iyz="0"
+          izz="1e-6"
+      />
+    </inertial>
+    <collision name='collision'>
+      <origin xyz="0 0 0" rpy="0 0 0"/>
+      <geometry>
+        <box size=".05 .05 .05"/>
+      </geometry>
+    </collision>
+    <visual name='camera_link_visual'>
+      <origin xyz="0 0 0" rpy="0 0 0"/>
+      <geometry>
+        <box size=".05 .05 .05"/>
+      </geometry>
+    </visual>
+  </link>
+  <gazebo reference="camera_link">
+    <material>Gazebo/Blue</material>
+  </gazebo>
+  <joint type="fixed" name="camera_optical_joint">
+    <origin xyz="0 0 0" rpy="-1.5707 0 -1.5707"/>
+    <child link="camera_link_optical"/>
+    <parent link="camera_link"/>
+  </joint>
+  <link name="camera_link_optical">
+  </link>
   </robot>

Commit message: Workin chess ai srv ,ikin ,trajectory
Still needs grabing mechanism

File: catkin_ws/src/ros_chess/urdf/chess_robot.xacro (robot description, xacro)
@@ -17,5 +17,5 @@
     <inertial>
       <mass value="5"/>
-      <origin xyz="0.0 0.0 0.0"/>
+      <origin xyz="0.0 0.0 0"/>
       <inertia ixx="0.1135" ixy="0.0" ixz="0.0"
                iyy="0.1135" iyz="0.0"
@@ -240,11 +240,11 @@
     <collision>
       <geometry>
-        <box size="0.1 0.01 0.2"/>
-      </geometry>
-      <origin xyz="0.0 0.0 0.0" rpy="0.0 0.0 0.0"/>
-    </collision>
-    <visual>
-      <geometry>
-        <box size="0.1 0.01 0.2"/>
+        <box size="0.0375 0.01 0.2"/>
+      </geometry>
+      <origin xyz="0.0 0.0 0.0" rpy="0.0 0.0 0.0"/>
+    </collision>
+    <visual>
+      <geometry>
+        <box size="0.0375 0.01 0.2"/>
       </geometry>
       <material name="blue"/>
@@ -282,11 +282,11 @@
     <collision>
       <geometry>
-        <box size="0.1 0.01 0.2"/>
-      </geometry>
-      <origin xyz="0.0 0.0 0.0" rpy="0.0 0.0 0.0"/>
-    </collision>
-    <visual>
-      <geometry>
-        <box size="0.1 0.01 0.2"/>
+        <box size="0.0375 0.01 0.2"/>
+      </geometry>
+      <origin xyz="0.0 0.0 0.0" rpy="0.0 0.0 0.0"/>
+    </collision>
+    <visual>
+      <geometry>
+        <box size="0.0375 0.01 0.2"/>
       </geometry>
       <material name="blue"/>
@@ -306,5 +306,5 @@
   <!--End effector (TCP) joint-->
   <joint name="end_effector_joint" type="fixed">
-    <origin xyz="0.0 0.0 0.175" rpy="0 0 0"/>
+    <origin xyz="0.0 0.0 0.2" rpy="0 0 0"/>
     <parent link="gripper_base_link"/>
     <child link="end_effector_link"/>

Commit message: Collada models
-minimal changes are needed

File: catkin_ws/src/ros_chess/urdf/chess_robot.xacro (robot description, xacro)
@@ -1,4 +1,4 @@
 <?xml version='1.0'?>
-<robot name="chess_arm" xmlns:xacro="http://www.ros.org/wiki/xacro">
+<robot name="chess_bot" xmlns:xacro="http://www.ros.org/wiki/xacro">
   <!-- RViz colors -->
   <xacro:include filename="$(find ros_chess)/urdf/materials.xacro" />
@@ -67,5 +67,8 @@
     <visual>
       <geometry>
+        <mesh filename = "package://ros_chess/gazebo_models/robot_arm/shoulder.dae"/>
+        <!--
         <cylinder radius="0.25" length="0.05"/>
+        -->
       </geometry>
       <material name="orange"/>
@@ -103,8 +106,11 @@
     <visual>
       <geometry>
+        <mesh filename = "package://ros_chess/gazebo_models/robot_arm/upper_arm.dae"/>
+        <!--
         <cylinder radius="0.1" length="1.5"/>
-      </geometry>
-      <material name="orange"/>
-      <origin xyz="0.0 0.0 0.75" rpy="0.0 0.0 0.0"/>
+        -->
+      </geometry>
+      <material name="orange"/>
+      <origin xyz="0.0 0.0 0.0" rpy="0.0 0.0 0.0"/>
     </visual>
   </link>
@@ -139,8 +145,11 @@
     <visual>
       <geometry>
+        <mesh filename = "package://ros_chess/gazebo_models/robot_arm/forearm.dae"/>
+        <!--
         <cylinder radius="0.10" length="1.5"/>
-      </geometry>
-      <material name="orange"/>
-      <origin xyz="0.0 0.0 0.75" rpy="0.0 0.0 0.0"/>
+        -->
+      </geometry>
+      <material name="orange"/>
+      <origin xyz="0.0 0.0 0.0" rpy="1.57079632679  0.0 0.0"/>
     </visual>
   </link>
@@ -175,8 +184,9 @@
     <visual>
       <geometry>
-        <cylinder radius="0.05" length="0.2"/>
-      </geometry>
-      <material name="orange"/>
-      <origin xyz="0.0 0.0 0.1" rpy="0.0 0.0 0.0"/>
+        <mesh filename = "package://ros_chess/gazebo_models/robot_arm/wrist.dae"/>
+        <!--<cylinder radius="0.05" length="0.2"/>-->
+      </geometry>
+      <material name="orange"/>
+      <origin xyz="-0.1 -0.15 0.15" rpy="0.0 0.0 0.0"/>
     </visual>
   </link>
@@ -211,8 +221,11 @@
     <visual>
       <geometry>
+        <mesh filename = "package://ros_chess/gazebo_models/robot_arm/gripper_base.dae"/>
+        <!--
         <box size=".1 .3 .02"/>
-      </geometry>
-      <material name="orange"/>
-      <origin xyz="0.0 0.0 0.01" rpy="0.0 0.0 0.0"/>
+        -->
+      </geometry>
+      <material name="orange"/>
+      <origin xyz="0.0 0.0 0.0" rpy="0.0 0.0 0.0"/>
     </visual>
   </link>
@@ -222,5 +235,5 @@
    <!-- Left finger joint -->
   <joint name="J6_left_finger_joint" type="prismatic">
-    <limit lower="0" upper="0.13" effort="50.0" velocity="4.0"/>
+    <limit lower="0" upper="0.05" effort="50.0" velocity="4.0"/>
     <parent link="gripper_base_link"/>
     <child link="left_finger"/>
@@ -232,5 +245,5 @@
     <inertial>
       <mass value="0.01"/>
-      <origin xyz="0.0 0.0 0.0" rpy="0.0 0.0 0.0"/>
+      <origin xyz="0.0 0.0 0.2" rpy="0.0 0.0 0.0"/>
       <inertia ixx="0.0009" ixy="0.0" ixz="0.0"
                iyy="0.0009" iyz="0.0"
@@ -248,5 +261,4 @@
         <box size="0.0375 0.01 0.2"/>
       </geometry>
-      <material name="blue"/>
       <origin xyz="0.0 0.0 0.0" rpy="0.0 0.0 0.0"/>
     </visual>
@@ -264,5 +276,5 @@
   <!-- Right finger joint -->
   <joint name="J7_right_finger_joint" type="prismatic">
-    <limit lower="0" upper="0.13" effort="50.0" velocity="4.0"/>
+    <limit lower="0" upper="0.05" effort="50.0" velocity="4.0"/>
     <parent link="gripper_base_link"/>
     <child link="right_finger"/>
@@ -274,5 +286,5 @@
     <inertial>
       <mass value="0.01"/>
-      <origin xyz="0.0 0.0 0.0" rpy="0.0 0.0 0.0"/>
+      <origin xyz="0.0 0.0 0.2" rpy="0.0 0.0 0.0"/>
       <inertia ixx="0.0009" ixy="0.0" ixz="0.0"
                iyy="0.0009" iyz="0.0"
@@ -290,5 +302,4 @@
         <box size="0.0375 0.01 0.2"/>
       </geometry>
-      <material name="blue"/>
       <origin xyz="0.0 0.0 0.0" rpy="0.0 0.0 0.0"/>
     </visual>
@@ -357,5 +368,5 @@
       <origin xyz="0 0 0" rpy="0 0 0"/>
       <geometry>
-        <box size=".05 .05 .05"/>
+        <box size=".04 .04 .045"/>
       </geometry>
     </visual>

Commit message: Functioning Robot
-This iteration has all the basic function witch is required for a working chess robot
-Additional chess move detections are needed (only) basic moves.

File: catkin_ws/src/ros_chess/urdf/chess_robot.xacro (robot description, xacro)
@@ -253,5 +253,5 @@
     <collision>
       <geometry>
-        <box size="0.0375 0.01 0.2"/>
+        <box size="0.02 0.015 0.2"/>
       </geometry>
       <origin xyz="0.0 0.0 0.0" rpy="0.0 0.0 0.0"/>
@@ -294,5 +294,5 @@
     <collision>
       <geometry>
-        <box size="0.0375 0.01 0.2"/>
+        <box size="0.02 0.005 0.1"/>
       </geometry>
       <origin xyz="0.0 0.0 0.0" rpy="0.0 0.0 0.0"/>
